Commit message: Depth check Done

File: mir_description/urdf/include/mir_250_v1.urdf.xacro (robot description, xacro)
@@ -44,5 +44,5 @@
   <!-- - 2x act wheels: 2kg -->
   <!--xacro:property name="mir_100_base_mass" value="66.96" /-->
-  <xacro:property name="mir_250_base_mass" value="97.0" />
+  <xacro:property name="mir_250_base_mass" value="200.0" />
   <xacro:property name="imu_stdev" value="0.00017" />
   <xacro:macro name="mir_250" params="prefix ns">
